Commit message: description: updating model with widowx arm

File: turtlebot_description/robots/kobuki_hexagons_astra_widowx.urdf.xacro (robot description, xacro)
@@ -12,5 +12,5 @@
   <sensor_astra parent="base_link"/>
   <widowx_arm parent="plate_top_link" prefix="">
-		<origin xyz="0.0 0.0 0.003" rpy="0.0 0.0 0.0"/>
+		<origin xyz="0.045 0.0 0.003" rpy="0.0 0.0 0.0"/>
   </widowx_arm>
 </robot>
