Commit message: Adding new sensor config and minor fixes

File: turtlebot_description/robots/kobuki_hexagons_astra_urg04lx.urdf.xacro (robot description, xacro)
@@ -4,5 +4,5 @@
     - Stacks    : hexagons
     - 3d Sensor : astra
-    - top_plate : widowx
+    - top_plate : urg04lx
 -->
 <robot name="turtlebot" xmlns:xacro="http://ros.org/wiki/xacro">
@@ -11,6 +11,6 @@
   <stack_hexagons parent="base_link"/>
   <sensor_astra parent="base_link"/>
-  <widowx_arm parent="plate_top_link" prefix="">
-		<origin xyz="0.0 0.0 0.003" rpy="0.0 0.0 0.0"/>
-  </widowx_arm>
+  <sensor_hokuyo_urg04lx name="hokuyo" parent="plate_top_link" >
+		<origin xyz="0.137 0 0.0525" rpy="0 0 0" />
+  </sensor_hokuyo_urg04lx>
 </robot>

File: turtlebot_description/robots/kobuki_hexagons_no3d_urg04lx.urdf.xacro (robot description, xacro)
@@ -3,5 +3,6 @@
     - Base      : kobuki
     - Stacks    : hexagons
-    - 3d Sensor : kinect
+    - 3d Sensor : no
+    - top_plate : urg04lx
 -->
 <robot name="turtlebot" xmlns:xacro="http://ros.org/wiki/xacro">

File: turtlebot_description/urdf/sensors/astra.urdf.xacro (robot description, xacro)
@@ -9,5 +9,5 @@
   <xacro:property name="astra_depth_rel_rgb_py" value="0.0250" />
   <xacro:property name="astra_cam_rel_rgb_py"   value="-0.0125" />
-  <xacro:property name="astra_dae_display_scale"   value="1" />
+  <xacro:property name="astra_dae_display_scale"   value="1.0" />
   <!-- Parameterised in part by the values in turtlebot_properties.urdf.xacro -->
   <xacro:macro name="sensor_astra" params="parent">

Commit message: updated to allow a multirobot system

File: turtlebot_description/robots/kobuki_hexagons_astra_urg04lx.urdf.xacro (robot description, xacro)
@@ -7,10 +7,12 @@
 -->
 <robot name="turtlebot" xmlns:xacro="http://ros.org/wiki/xacro">
-  <xacro:include filename="$(find turtlebot_description)/urdf/turtlebot_library.urdf.xacro" />
-  <kobuki/>
-  <stack_hexagons parent="base_link"/>
-  <sensor_astra parent="base_link"/>
-  <sensor_hokuyo_urg04lx name="hokuyo" parent="plate_top_link" >
+  <xacro:arg name="prefix_frame" default=""/>
+  <xacro:include filename="$(find turtlebot_description)/urdf/turtlebot_library_multi.urdf.xacro" />
+  <xacro:kobuki prefix_frame="$(arg prefix_frame)"/>
+  <xacro:stack_hexagons prefix_frame="$(arg prefix_frame)"  parent="$(arg prefix_frame)base_link"/>
+  <xacro:sensor_astra prefix_frame="$(arg prefix_frame)" parent="$(arg prefix_frame)base_link"/>
+  <xacro:sensor_hokuyo_urg04lx name="hokuyo" prefix_frame="$(arg prefix_frame)" parent="$(arg prefix_frame)plate_top_link" >
 		<origin xyz="0.137 0 0.0525" rpy="0 0 0" />
-  </sensor_hokuyo_urg04lx>
+  </xacro:sensor_hokuyo_urg04lx>
+  <!-- here add the arm -->
 </robot>

File: turtlebot_description/urdf/sensors/astra.urdf.xacro (robot description, xacro)
@@ -9,25 +9,25 @@
   <xacro:property name="astra_dae_display_scale"   value="1.0" />
   <!-- Parameterised in part by the values in turtlebot_properties.urdf.xacro -->
-  <xacro:macro name="sensor_astra" params="parent">
-    <joint name="camera_rgb_joint" type="fixed">
+  <xacro:macro name="sensor_astra" params="prefix_frame parent">
+    <joint name="${prefix_frame}camera_rgb_joint" type="fixed">
       <origin xyz="${cam_px} ${astra_cam_py} ${cam_pz}"
               rpy="0 0 0"/>
       <parent link="${parent}"/>
-      <child link="camera_rgb_frame" />
+      <child link="${prefix_frame}camera_rgb_frame" />
     </joint>
-    <link name="camera_rgb_frame"/>
-    <joint name="camera_rgb_optical_joint" type="fixed">
+    <link name="${prefix_frame}camera_rgb_frame"/>
+    <joint name="${prefix_frame}camera_rgb_optical_joint" type="fixed">
       <origin xyz="0 0 0" rpy="${-M_PI/2} 0 ${-M_PI/2}" />
-      <parent link="camera_rgb_frame" />
-      <child link="camera_rgb_optical_frame" />
+      <parent link="${prefix_frame}camera_rgb_frame" />
+      <child link="${prefix_frame}camera_rgb_optical_frame" />
     </joint>
-    <link name="camera_rgb_optical_frame"/>
-    <joint name="camera_joint" type="fixed">
+    <link name="${prefix_frame}camera_rgb_optical_frame"/>
+    <joint name="${prefix_frame}camera_joint" type="fixed">
       <origin xyz="0 ${astra_cam_rel_rgb_py} 0"
               rpy="0 0 0"/>
-      <parent link="camera_rgb_frame"/>
-      <child link="camera_link"/>
+      <parent link="${prefix_frame}camera_rgb_frame"/>
+      <child link="${prefix_frame}camera_link"/>
     </joint>
-    <link name="camera_link">
+    <link name="${prefix_frame}camera_link">
       <visual>
         <origin xyz="0 0 0" rpy="0 0 0"/>
@@ -50,18 +50,18 @@
       </inertial>
     </link>
-    <joint name="camera_depth_joint" type="fixed">
+    <joint name="${prefix_frame}camera_depth_joint" type="fixed">
       <origin xyz="0 ${astra_depth_rel_rgb_py} 0" rpy="0 0 0" />
-      <parent link="camera_rgb_frame" />
-      <child link="camera_depth_frame" />
+      <parent link="${prefix_frame}camera_rgb_frame" />
+      <child link="${prefix_frame}camera_depth_frame" />
     </joint>
-    <link name="camera_depth_frame"/>
-    <joint name="camera_depth_optical_joint" type="fixed">
+    <link name="${prefix_frame}camera_depth_frame"/>
+    <joint name="${prefix_frame}camera_depth_optical_joint" type="fixed">
       <origin xyz="0 0 0" rpy="${-M_PI/2} 0 ${-M_PI/2}" />
-      <parent link="camera_depth_frame" />
-      <child link="camera_depth_optical_frame" />
+      <parent link="${prefix_frame}camera_depth_frame" />
+      <child link="${prefix_frame}camera_depth_optical_frame" />
     </joint>
-    <link name="camera_depth_optical_frame"/>
+    <link name="${prefix_frame}camera_depth_optical_frame"/>
     <!-- RGBD sensor for simulation, same as Kinect -->
-    <turtlebot_sim_3dsensor/>
+    <turtlebot_sim_3dsensor prefix_frame="${prefix_frame}"/>
   </xacro:macro>
 </robot>

File: turtlebot_description/urdf/sensors/hokuyo_urg04lx.urdf.xacro (robot description, xacro)
@@ -2,15 +2,15 @@
 <robot name="sensor_hokuyo_urg04lx" xmlns:xacro="http://ros.org/wiki/xacro">
   <xacro:property name="H_SCALE" value="0.025"/>
-  <xacro:macro name="sensor_hokuyo_urg04lx" params="name parent *origin min_angle:=2.0943 max_angle:=-2.0943">
-    <joint name="${name}_laser_joint" type="fixed">
+  <xacro:macro name="sensor_hokuyo_urg04lx" params="name prefix_frame parent *origin min_angle:=2.0943 max_angle:=-2.0943">
+    <joint name="${prefix_frame}${name}_laser_joint" type="fixed">
       <!-- FRONT MOUNT  -->
       <!-- origin xyz="0.29 0 0.1" -->
       <!-- TOP MOUNT -->
       <!-- origin xyz="0.0 0.0 0.325"-->
-      <insert_block name="origin" />
+      <xacro:insert_block name="origin" />
       <parent link="${parent}"/>
-      <child link="${name}_laser_link"/>
+      <child link="${prefix_frame}${name}_laser_link"/>
     </joint>
-    <link name="${name}_laser_link">
+    <link name="${prefix_frame}${name}_laser_link">
       <collision>
         <origin xyz="0 0 -0.05" rpy="0 0 0"/>
@@ -32,8 +32,8 @@
     </link>
     <!-- Hokuyo sensor for simulation -->
-    <sensor_hokuyo_urg_gazebo/>
+    <xacro:sensor_hokuyo_urg_gazebo prefix_frame="${prefix_frame}"/>
   </xacro:macro>
-  <xacro:macro name="sensor_hokuyo_urg_gazebo">
-    <gazebo reference="${name}_laser_link">
+  <xacro:macro name="sensor_hokuyo_urg_gazebo" params="prefix_frame">
+    <gazebo reference="${prefix_frame}${name}_laser_link">
 			<sensor type="ray" name="${name}_sensor">
 				<pose>0 0 0 0 0 0</pose>
@@ -62,5 +62,6 @@
 				<plugin name="gazebo_ros_head_hokuyo_controller" filename="libgazebo_ros_laser.so">
 					<topicName>${name}/scan</topicName>
-					<frameName>${name}_laser_link</frameName>
+					<frameName>${prefix_frame}${name}_laser_link</frameName>
+					<ignoreTfPrefix>1</ignoreTfPrefix>
 				</plugin>
 			</sensor>

File: turtlebot_description/urdf/sensors/rplidar.urdf.xacro (robot description, xacro)
@@ -3,5 +3,5 @@
   <xacro:macro name="sensor_rplidar" params="prefix parent *origin min_angle:=3.14159 max_angle:=-3.14159">
     <joint name="${prefix}_laser_base_joint" type="fixed">
-      <insert_block name="origin" />
+      <xacro:insert_block name="origin" />
       <parent link="${parent}"/>
       <child link="${prefix}_laser_base_link"/>

File: turtlebot_description/urdf/stacks/hexagons.urdf.xacro (robot description, xacro)
@@ -9,11 +9,11 @@
   <!-- Xacro macros -->
   <!-- Pole macros -->
-  <xacro:macro name="stack_bottom_pole" params="parent number x_loc y_loc z_loc">
-    <joint name="pole_bottom_${number}_joint" type="fixed">
+  <xacro:macro name="stack_bottom_pole" params="prefix_frame parent number x_loc y_loc z_loc">
+    <joint name="${prefix_frame}pole_bottom_${number}_joint" type="fixed">
       <origin xyz="${x_loc} ${y_loc} ${z_loc}" rpy="0 0 0"/>
       <parent link="${parent}"/>
-      <child link="pole_bottom_${number}_link"/>
-    </joint>
-    <link name="pole_bottom_${number}_link">
+      <child link="${prefix_frame}pole_bottom_${number}_link"/>
+    </joint>
+    <link name="${prefix_frame}pole_bottom_${number}_link">
       <visual>
         <origin xyz="0 0 0" rpy="0 0 0"/>
@@ -37,11 +37,11 @@
     </link>
   </xacro:macro>
-  <xacro:macro name="stack_middle_pole" params="parent number x_loc y_loc z_loc">
-    <joint name="pole_middle_${number}_joint" type="fixed">
+  <xacro:macro name="stack_middle_pole" params="prefix_frame parent number x_loc y_loc z_loc">
+    <joint name="${prefix_frame}pole_middle_${number}_joint" type="fixed">
       <origin xyz="${x_loc} ${y_loc} ${z_loc}" rpy="0 0 0" />
       <parent link="${parent}"/>
-      <child link="pole_middle_${number}_link"/>
-    </joint>
-    <link name="pole_middle_${number}_link">
+      <child link="${prefix_frame}pole_middle_${number}_link"/>
+    </joint>
+    <link name="${prefix_frame}pole_middle_${number}_link">
       <visual>
         <origin xyz="0 0 0" rpy="0 ${M_PI} 0"/>
@@ -65,11 +65,11 @@
     </link>
   </xacro:macro>
-  <xacro:macro name="stack_top_pole" params="parent number x_loc y_loc z_loc">
-    <joint name="pole_top_${number}_joint" type="fixed">
+  <xacro:macro name="stack_top_pole" params="prefix_frame parent number x_loc y_loc z_loc">
+    <joint name="${prefix_frame}pole_top_${number}_joint" type="fixed">
       <origin xyz="${x_loc} ${y_loc} ${z_loc}" rpy="0 0 0"/>
       <parent link="${parent}"/>
-      <child link="pole_top_${number}_link"/>
-    </joint>
-    <link name="pole_top_${number}_link">
+      <child link="${prefix_frame}pole_top_${number}_link"/>
+    </joint>
+    <link name="${prefix_frame}pole_top_${number}_link">
       <visual>
         <origin xyz=" 0 0 0" rpy="0 0 0"/>
@@ -93,11 +93,11 @@
     </link>
   </xacro:macro>
-  <xacro:macro name="stack_3d_sensor_pole" params="parent number x_loc y_loc z_loc">
-    <joint name="pole_kinect_${number}_joint" type="fixed">
+  <xacro:macro name="stack_3d_sensor_pole" params="prefix_frame parent number x_loc y_loc z_loc">
+    <joint name="${prefix_frame}pole_kinect_${number}_joint" type="fixed">
       <origin xyz="${x_loc} ${y_loc} ${z_loc}" rpy="0 0 0"/>
       <parent link="${parent}"/>
-      <child link="pole_kinect_${number}_link"/>
-    </joint>
-    <link name="pole_kinect_${number}_link">
+      <child link="${prefix_frame}pole_kinect_${number}_link"/>
+    </joint>
+    <link name="${prefix_frame}pole_kinect_${number}_link">
       <visual>
         <origin xyz="0 0 -0.01" rpy="0 0 0"/>
@@ -126,17 +126,17 @@
     other, but there is no necessary reason to do so.
   -->
-  <xacro:macro name="stack_hexagons" params="parent">
-    <stack_bottom_pole parent="${parent}" number="0" x_loc= "0.120" y_loc= "0.082" z_loc="0.1028"/>
-    <stack_bottom_pole parent="${parent}" number="1" x_loc= "0.055" y_loc= "0.120" z_loc="0.1028"/>
-    <stack_bottom_pole parent="${parent}" number="2" x_loc="-0.055" y_loc= "0.120" z_loc="0.1028"/>
-    <stack_bottom_pole parent="${parent}" number="3" x_loc= "0.120" y_loc="-0.082" z_loc="0.1028"/>
-    <stack_bottom_pole parent="${parent}" number="4" x_loc= "0.055" y_loc="-0.120" z_loc="0.1028"/>
-    <stack_bottom_pole parent="${parent}" number="5" x_loc="-0.055" y_loc="-0.120" z_loc="0.1028"/>
-    <joint name="plate_bottom_joint" type="fixed">
+  <xacro:macro name="stack_hexagons" params="prefix_frame parent">
+    <stack_bottom_pole prefix_frame="${prefix_frame}" parent="${parent}" number="0" x_loc= "0.120" y_loc= "0.082" z_loc="0.1028"/>
+    <stack_bottom_pole prefix_frame="${prefix_frame}" parent="${parent}" number="1" x_loc= "0.055" y_loc= "0.120" z_loc="0.1028"/>
+    <stack_bottom_pole prefix_frame="${prefix_frame}" parent="${parent}" number="2" x_loc="-0.055" y_loc= "0.120" z_loc="0.1028"/>
+    <stack_bottom_pole prefix_frame="${prefix_frame}" parent="${parent}" number="3" x_loc= "0.120" y_loc="-0.082" z_loc="0.1028"/>
+    <stack_bottom_pole prefix_frame="${prefix_frame}" parent="${parent}" number="4" x_loc= "0.055" y_loc="-0.120" z_loc="0.1028"/>
+    <stack_bottom_pole prefix_frame="${prefix_frame}" parent="${parent}" number="5" x_loc="-0.055" y_loc="-0.120" z_loc="0.1028"/>
+    <joint name="${prefix_frame}plate_bottom_joint" type="fixed">
       <origin xyz="0.02364 0.0 0.1306" rpy="0 0 0"/>
       <parent link="${parent}"/>
-      <child link="plate_bottom_link"/>
-    </joint>
-    <link name="plate_bottom_link">
+      <child link="${prefix_frame}plate_bottom_link"/>
+    </joint>
+    <link name="${prefix_frame}plate_bottom_link">
       <visual>
         <origin xyz="0 0 0" rpy="0 0 0"/>
@@ -159,14 +159,14 @@
       </inertial>
     </link>
-    <stack_middle_pole parent="${parent}" number="0" x_loc= "0.0381" y_loc= "0.1505" z_loc="0.1640"/>
-    <stack_middle_pole parent="${parent}" number="1" x_loc= "0.0381" y_loc="-0.1505" z_loc="0.1640"/>
-    <stack_middle_pole parent="${parent}" number="2" x_loc="-0.0381" y_loc= "0.1505" z_loc="0.1640"/>
-    <stack_middle_pole parent="${parent}" number="3" x_loc="-0.0381" y_loc="-0.1505" z_loc="0.1640"/>
-    <joint name="plate_middle_joint" type="fixed">
+    <stack_middle_pole prefix_frame="${prefix_frame}" parent="${parent}" number="0" x_loc= "0.0381" y_loc= "0.1505" z_loc="0.1640"/>
+    <stack_middle_pole prefix_frame="${prefix_frame}" parent="${parent}" number="1" x_loc= "0.0381" y_loc="-0.1505" z_loc="0.1640"/>
+    <stack_middle_pole prefix_frame="${prefix_frame}" parent="${parent}" number="2" x_loc="-0.0381" y_loc= "0.1505" z_loc="0.1640"/>
+    <stack_middle_pole prefix_frame="${prefix_frame}" parent="${parent}" number="3" x_loc="-0.0381" y_loc="-0.1505" z_loc="0.1640"/>
+    <joint name="${prefix_frame}plate_middle_joint" type="fixed">
       <origin xyz="-0.01364 0.0 0.1874" rpy="0 0 0"/>
       <parent link="${parent}"/>
-      <child link="plate_middle_link"/>
-    </joint>
-    <link name="plate_middle_link">
+      <child link="${prefix_frame}plate_middle_link"/>
+    </joint>
+    <link name="${prefix_frame}plate_middle_link">
       <visual>
         <origin xyz="0 0 0" rpy="0 0 0"/>
@@ -189,16 +189,16 @@
       </inertial>
     </link>
-    <stack_top_pole parent="${parent}" number="0" x_loc= "0.0381" y_loc= "0.1505" z_loc="0.2920"/>
-    <stack_top_pole parent="${parent}" number="1" x_loc= "0.0381" y_loc="-0.1505" z_loc="0.2920"/>
-    <stack_top_pole parent="${parent}" number="2" x_loc="-0.0381" y_loc= "0.1505" z_loc="0.2920"/>
-    <stack_top_pole parent="${parent}" number="3" x_loc="-0.0381" y_loc="-0.1505" z_loc="0.2920"/>
-    <stack_3d_sensor_pole parent="${parent}" number="0" x_loc="-0.1024" y_loc= "0.098" z_loc="0.2372"/>
-    <stack_3d_sensor_pole parent="${parent}" number="1" x_loc="-0.1024" y_loc="-0.098" z_loc="0.2372"/>
-    <joint name="plate_top_joint" type="fixed">
+    <stack_top_pole prefix_frame="${prefix_frame}" parent="${parent}" number="0" x_loc= "0.0381" y_loc= "0.1505" z_loc="0.2920"/>
+    <stack_top_pole prefix_frame="${prefix_frame}" parent="${parent}" number="1" x_loc= "0.0381" y_loc="-0.1505" z_loc="0.2920"/>
+    <stack_top_pole prefix_frame="${prefix_frame}" parent="${parent}" number="2" x_loc="-0.0381" y_loc= "0.1505" z_loc="0.2920"/>
+    <stack_top_pole prefix_frame="${prefix_frame}" parent="${parent}" number="3" x_loc="-0.0381" y_loc="-0.1505" z_loc="0.2920"/>
+    <stack_3d_sensor_pole prefix_frame="${prefix_frame}" parent="${parent}" number="0" x_loc="-0.1024" y_loc= "0.098" z_loc="0.2372"/>
+    <stack_3d_sensor_pole prefix_frame="${prefix_frame}" parent="${parent}" number="1" x_loc="-0.1024" y_loc="-0.098" z_loc="0.2372"/>
+    <joint name="${prefix_frame}plate_top_joint" type="fixed">
       <origin xyz="-0.01364 0.0  0.3966" rpy="0 0 0"/>
       <parent link="${parent}"/>
-      <child link="plate_top_link"/>
-    </joint>
-    <link name="plate_top_link">
+      <child link="${prefix_frame}plate_top_link"/>
+    </joint>
+    <link name="${prefix_frame}plate_top_link">
       <visual>
         <origin xyz="0 0 0" rpy="0 0 0"/>

File: turtlebot_description/urdf/turtlebot_gazebo.urdf.xacro (robot description, xacro)
@@ -2,6 +2,6 @@
 <robot name="turtlebot_gazebo" xmlns:xacro="http://ros.org/wiki/xacro">
   <!-- Microsoft Kinect / ASUS Xtion PRO Live for simulation -->
-  <xacro:macro name="turtlebot_sim_3dsensor">
-    <gazebo reference="camera_link">
+  <xacro:macro name="turtlebot_sim_3dsensor" params="prefix_frame">
+    <gazebo reference="${prefix_frame}camera_link">
       <sensor type="depth" name="camera">
         <always_on>true</always_on>
@@ -28,5 +28,5 @@
           <cameraInfoTopicName>rgb/camera_info</cameraInfoTopicName>
           <depthImageCameraInfoTopicName>depth/camera_info</depthImageCameraInfoTopicName>
-          <frameName>camera_depth_optical_frame</frameName>
+          <frameName>${prefix_frame}camera_depth_optical_frame</frameName>
           <baseline>0.1</baseline>
           <distortion_k1>0.0</distortion_k1>
@@ -35,4 +35,5 @@
           <distortion_t1>0.0</distortion_t1>
           <distortion_t2>0.0</distortion_t2>
+          <ignoreTfPrefix>1</ignoreTfPrefix>
           <pointCloudCutoff>0.4</pointCloudCutoff>
         </plugin>
