Commit message: xacro changes to add the prefix_frame

File: turtlebot_description/robots/kobuki_hexagons_astra_urg04lx.urdf.xacro (robot description, xacro)
@@ -12,7 +12,7 @@
   <xacro:stack_hexagons prefix_frame="$(arg prefix_frame)"  parent="$(arg prefix_frame)base_link"/>
   <xacro:sensor_astra prefix_frame="$(arg prefix_frame)" parent="$(arg prefix_frame)base_link"/>
-  <xacro:sensor_hokuyo_urg04lx name="hokuyo" prefix_frame="$(arg prefix_frame)" parent="$(arg prefix_frame)plate_top_link" >
+  <sensor_hokuyo_urg04lx prefix="$(arg prefix_frame)" parent="$(arg prefix_frame)plate_top_link" >
 		<origin xyz="0.137 0 0.0525" rpy="0 0 0" />
-  </xacro:sensor_hokuyo_urg04lx>
+  </sensor_hokuyo_urg04lx>
   <!-- here add the arm -->
 </robot>

File: turtlebot_description/robots/kobuki_hexagons_kinect_.urdf.xacro (robot description, xacro)
@@ -6,10 +6,12 @@
 -->
 <robot name="turtlebot" xmlns:xacro="http://ros.org/wiki/xacro">
-  <xacro:include filename="$(find turtlebot_description)/urdf/turtlebot_common_library.urdf.xacro" />
-  <xacro:include filename="$(find kobuki_description)/urdf/kobuki.urdf.xacro" />
+  <xacro:arg name="prefix_frame" default=""/>
+  <!--xacro:include filename="$(find turtlebot_description)/urdf/turtlebot_common_library.urdf.xacro" /-->
+  <xacro:include filename="$(find turtlebot_description)/urdf/turtlebot_library_multi.urdf.xacro" />
+  <!--xacro:include filename="$(find kobuki_description)/urdf/kobuki.urdf.xacro" /-->
   <xacro:include filename="$(find turtlebot_description)/urdf/stacks/hexagons.urdf.xacro"/>
   <xacro:include filename="$(find turtlebot_description)/urdf/sensors/kinect.urdf.xacro"/>
-  <kobuki/>
-  <stack_hexagons parent="base_link"/>
-  <sensor_kinect  parent="base_link"/>
+  <kobuki prefix_frame="$(arg prefix_frame)"/>
+  <stack_hexagons prefix_frame="$(arg prefix_frame)" parent="$(arg prefix_frame)base_link"/>
+  <sensor_kinect prefix_frame="$(arg prefix_frame)" parent="$(arg prefix_frame)base_link"/>
 </robot>

File: turtlebot_description/robots/kobuki_hexagons_no3d_urg04lx.urdf.xacro (robot description, xacro)
@@ -7,8 +7,11 @@
 -->
 <robot name="turtlebot" xmlns:xacro="http://ros.org/wiki/xacro">
-  <xacro:include filename="$(find turtlebot_description)/urdf/turtlebot_library.urdf.xacro" />
-  <kobuki/>
-  <stack_hexagons parent="base_link"/>
-  <sensor_hokuyo_urg04lx name="hokuyo" parent="plate_top_link" >
+  <xacro:arg name="prefix_frame" default=""/>
+  <!--xacro:include filename="$(find turtlebot_description)/urdf/turtlebot_library.urdf.xacro" /-->
+  <xacro:include filename="$(find turtlebot_description)/urdf/turtlebot_library_multi.urdf.xacro" />
+  <xacro:include filename="$(find turtlebot_description)/urdf/stacks/hexagons.urdf.xacro"/>
+  <kobuki prefix_frame="$(arg prefix_frame)"/>
+  <stack_hexagons prefix_frame="$(arg prefix_frame)" parent="$(arg prefix_frame)base_link"/>
+  <sensor_hokuyo_urg04lx prefix="$(arg prefix_frame)" parent="$(arg prefix_frame)plate_top_link" >
 		<origin xyz="0.137 0 0.0525" rpy="0 0 0" />
   </sensor_hokuyo_urg04lx>

File: turtlebot_description/urdf/sensors/hokuyo_urg04lx.urdf.xacro (robot description, xacro)
@@ -2,6 +2,7 @@
 <robot name="sensor_hokuyo_urg04lx" xmlns:xacro="http://ros.org/wiki/xacro">
   <xacro:property name="H_SCALE" value="0.025"/>
-  <xacro:macro name="sensor_hokuyo_urg04lx" params="name prefix_frame parent *origin min_angle:=2.0943 max_angle:=-2.0943">
-    <joint name="${prefix_frame}${name}_laser_joint" type="fixed">
+  <!--xacro:macro name="sensor_hokuyo_urg04lx" params="prefix parent *origin min_angle:=2.0943 max_angle:=-2.0943"-->
+  <xacro:macro name="sensor_hokuyo_urg04lx" params="prefix parent *origin min_angle:=1.59 max_angle:=-1.59">
+    <joint name="${prefix}laser_joint" type="fixed">
       <!-- FRONT MOUNT  -->
       <!-- origin xyz="0.29 0 0.1" -->
@@ -10,7 +11,7 @@
       <xacro:insert_block name="origin" />
       <parent link="${parent}"/>
-      <child link="${prefix_frame}${name}_laser_link"/>
+      <child link="${prefix}laser_link"/>
     </joint>
-    <link name="${prefix_frame}${name}_laser_link">
+    <link name="${prefix}laser_link">
       <collision>
         <origin xyz="0 0 -0.05" rpy="0 0 0"/>
@@ -32,9 +33,9 @@
     </link>
     <!-- Hokuyo sensor for simulation -->
-    <xacro:sensor_hokuyo_urg_gazebo prefix_frame="${prefix_frame}"/>
+    <xacro:sensor_hokuyo_urg_gazebo prefix="${prefix}"/>
   </xacro:macro>
-  <xacro:macro name="sensor_hokuyo_urg_gazebo" params="prefix_frame">
-    <gazebo reference="${prefix_frame}${name}_laser_link">
-			<sensor type="ray" name="${name}_sensor">
+  <xacro:macro name="sensor_hokuyo_urg_gazebo" params="prefix">
+    <gazebo reference="${prefix}laser_link">
+			<sensor type="ray" name="${prefix}sensor">
 				<pose>0 0 0 0 0 0</pose>
 				<visualize>false</visualize>
@@ -61,6 +62,6 @@
 				</ray>
 				<plugin name="gazebo_ros_head_hokuyo_controller" filename="libgazebo_ros_laser.so">
-					<topicName>${name}/scan</topicName>
-					<frameName>${prefix_frame}${name}_laser_link</frameName>
+					<topicName>scan</topicName>
+					<frameName>${prefix}laser_link</frameName>
 					<ignoreTfPrefix>1</ignoreTfPrefix>
 				</plugin>

File: turtlebot_description/urdf/sensors/kinect.urdf.xacro (robot description, xacro)
@@ -5,23 +5,23 @@
   <xacro:property name="kinect_cam_py" value="-0.0125"/>
   <!-- Parameterised in part by the values in turtlebot_properties.urdf.xacro -->
-  <xacro:macro name="sensor_kinect" params="parent">
-    <joint name="camera_rgb_joint" type="fixed">
+  <xacro:macro name="sensor_kinect" params="prefix_frame parent">
+    <joint name="${prefix_frame}camera_rgb_joint" type="fixed">
       <origin xyz="${cam_px} ${kinect_cam_py} ${cam_pz}" rpy="${cam_or} ${cam_op} ${cam_oy}"/>
       <parent link="${parent}"/>
-      <child link="camera_rgb_frame" />
+      <child link="${prefix_frame}camera_rgb_frame" />
     </joint>
-    <link name="camera_rgb_frame"/>
-    <joint name="camera_rgb_optical_joint" type="fixed">
+    <link name="${prefix_frame}camera_rgb_frame"/>
+    <joint name="${prefix_frame}camera_rgb_optical_joint" type="fixed">
       <origin xyz="0 0 0" rpy="${-M_PI/2} 0 ${-M_PI/2}" />
-      <parent link="camera_rgb_frame" />
-      <child link="camera_rgb_optical_frame" />
+      <parent link="${prefix_frame}camera_rgb_frame" />
+      <child link="${prefix_frame}camera_rgb_optical_frame" />
     </joint>
-    <link name="camera_rgb_optical_frame"/>
-    <joint name="camera_joint" type="fixed">
+    <link name="${prefix_frame}camera_rgb_optical_frame"/>
+    <joint name="${prefix_frame}camera_joint" type="fixed">
       <origin xyz="-0.031 ${-kinect_cam_py} -0.016" rpy="0 0 0"/>
-      <parent link="camera_rgb_frame"/>
-      <child link="camera_link"/>
+      <parent link="${prefix_frame}camera_rgb_frame"/>
+      <child link="${prefix_frame}camera_link"/>
     </joint>
-      <link name="camera_link">
+      <link name="${prefix_frame}camera_link">
       <visual>
        <origin xyz="0 0 0" rpy="0 0 ${M_PI/2}"/>
@@ -47,18 +47,18 @@
          files. However, for Gazebo simulation we need them, so we add them here.
          (Hence, don't publish them additionally!) -->
-	<joint name="camera_depth_joint" type="fixed">
+	<joint name="${prefix_frame}camera_depth_joint" type="fixed">
 	  <origin xyz="0 ${2 * -kinect_cam_py} 0" rpy="0 0 0" />
-	  <parent link="camera_rgb_frame" />
-	  <child link="camera_depth_frame" />
+	  <parent link="${prefix_frame}camera_rgb_frame" />
+	  <child link="${prefix_frame}camera_depth_frame" />
 	</joint>
-	<link name="camera_depth_frame"/>
-	<joint name="camera_depth_optical_joint" type="fixed">
+	<link name="${prefix_frame}camera_depth_frame"/>
+	<joint name="${prefix_frame}camera_depth_optical_joint" type="fixed">
 	  <origin xyz="0 0 0" rpy="${-M_PI/2} 0 ${-M_PI/2}" />
-	  <parent link="camera_depth_frame" />
-	  <child link="camera_depth_optical_frame" />
+	  <parent link="${prefix_frame}camera_depth_frame" />
+	  <child link="${prefix_frame}camera_depth_optical_frame" />
 	</joint>
-	<link name="camera_depth_optical_frame"/>
+	<link name="${prefix_frame}camera_depth_optical_frame"/>
 	<!-- Kinect sensor for simulation -->
-	<turtlebot_sim_3dsensor/>
+	<turtlebot_sim_3dsensor prefix_frame="${prefix_frame}"/>
   </xacro:macro>
 </robot>
