Commit message: added rplidar sensor

File: turtlebot_description/robots/kobuki_hexagons_no3d_rplidar.urdf.xacro (robot description, xacro)
@@ -6,8 +6,9 @@
 -->
 <robot name="turtlebot" xmlns:xacro="http://ros.org/wiki/xacro">
-  <xacro:include filename="$(find turtlebot_description)/urdf/turtlebot_library.urdf.xacro" />
-  <kobuki/>
-  <stack_hexagons parent="base_link"/>
-  <sensor_rplidar  parent="plate_top_link" prefix="rplidar">
+  <xacro:arg name="prefix_frame" default=""/>
+  <xacro:include filename="$(find turtlebot_description)/urdf/turtlebot_library_multi.urdf.xacro" />
+  <xacro:kobuki prefix_frame="$(arg prefix_frame)"/>
+  <xacro:stack_hexagons prefix_frame="$(arg prefix_frame)"  parent="$(arg prefix_frame)base_link"/>
+  <sensor_rplidar prefix="$(arg prefix_frame)" parent="$(arg prefix_frame)plate_top_link">
 	<origin xyz="0 0.0 0.005" rpy="0 0 0"/>
   </sensor_rplidar>

File: turtlebot_description/urdf/sensors/rplidar.urdf.xacro (robot description, xacro)
@@ -2,14 +2,14 @@
 <robot xmlns:xacro="http://ros.org/wiki/xacro">
   <xacro:macro name="sensor_rplidar" params="prefix parent *origin min_angle:=3.14159 max_angle:=-3.14159">
-    <joint name="${prefix}_laser_base_joint" type="fixed">
+    <joint name="${prefix}laser_base_joint" type="fixed">
       <xacro:insert_block name="origin" />
       <parent link="${parent}"/>
-      <child link="${prefix}_laser_base_link"/>
+      <child link="${prefix}laser_base_link"/>
     </joint>
-    <link name="${prefix}_laser_base_link">
+    <link name="${prefix}laser_base_link">
       <collision>
         <origin xyz="0 0 0" rpy="0 0 0"/>
         <geometry>
-            <mesh filename="package://turtlebot_description/meshes/sensors/rplidar.dae"/>
+            <mesh filename="package://turtlebot_description/meshes/sensors/rplidar.stl"/>
         </geometry>
       </collision>
@@ -26,16 +26,16 @@
       </inertial>
     </link>
-    <joint name="${prefix}_laser_joint" type="fixed">
+    <joint name="${prefix}laser_joint" type="fixed">
       <origin xyz="0 0 0.0461" rpy="0 0 0"/>
-      <parent link="${prefix}_laser_base_link"/>
-      <child link="${prefix}_laser_link"/>
+      <parent link="${prefix}laser_base_link"/>
+      <child link="${prefix}laser_link"/>
     </joint>
-    <link name="${prefix}_laser_link">
+    <link name="${prefix}laser_link">
     </link>
     <sensor_rplidar_gazebo/>
   </xacro:macro>
   <xacro:macro name="sensor_rplidar_gazebo">
-    <gazebo reference="${prefix}_laser_link">
-			<sensor type="ray" name="${prefix}_rplidar_sensor">
+    <gazebo reference="${prefix}laser_link">
+			<sensor type="ray" name="${prefix}rplidar_sensor">
 				<pose>0 0 0 0 0 0</pose>
 				<visualize>false</visualize>
@@ -62,6 +62,7 @@
 				</ray>
 				<plugin name="gazebo_ros_rplidar_controller" filename="libgazebo_ros_laser.so">
-					<topicName>${prefix}/scan</topicName>
-					<frameName>${prefix}_laser_link</frameName>
+					<topicName>scan</topicName>
+					<frameName>${prefix}laser_link</frameName>
+					<ignoreTfPrefix>1</ignoreTfPrefix>
 				</plugin>
 			</sensor>

File: turtlebot_description/urdf/turtlebot_library_multi.urdf.xacro (robot description, xacro)
@@ -8,5 +8,5 @@
   <xacro:include filename="$(find turtlebot_description)/urdf/turtlebot_properties.urdf.xacro"/>
   <!-- Bases -->
-  <xacro:include filename="$(find create_description)/urdf/create.urdf.xacro"/>
+  <!--xacro:include filename="$(find create_description)/urdf/create.urdf.xacro"/-->
   <xacro:include filename="$(find turtlebot_description)/urdf/kobuki_multi.urdf.xacro" />
   <!-- Stacks -->
