Commit message: limited the range of hokuyo_urg04lx

File: turtlebot_description/urdf/sensors/hokuyo_urg04lx.urdf.xacro (robot description, xacro)
@@ -3,5 +3,5 @@
   <xacro:property name="H_SCALE" value="0.025"/>
   <!--xacro:macro name="sensor_hokuyo_urg04lx" params="prefix parent *origin min_angle:=2.0943 max_angle:=-2.0943"-->
-  <xacro:macro name="sensor_hokuyo_urg04lx" params="prefix parent *origin min_angle:=1.59 max_angle:=-1.59">
+  <xacro:macro name="sensor_hokuyo_urg04lx" params="prefix parent *origin min_angle:=1.5708 max_angle:=-1.5708">
     <joint name="${prefix}laser_joint" type="fixed">
       <!-- FRONT MOUNT  -->
@@ -44,5 +44,6 @@
 					<scan>
 						<horizontal>
-							<samples>681</samples>
+							<!--samples>681</samples-->
+							<samples>180</samples>
 							<resolution>1</resolution>
 							<min_angle>${min_angle}</min_angle>

Commit message: modified the range of the laser

File: turtlebot_description/urdf/sensors/hokuyo_urg04lx.urdf.xacro (robot description, xacro)
@@ -3,5 +3,6 @@
   <xacro:property name="H_SCALE" value="0.025"/>
   <!--xacro:macro name="sensor_hokuyo_urg04lx" params="prefix parent *origin min_angle:=2.0943 max_angle:=-2.0943"-->
-  <xacro:macro name="sensor_hokuyo_urg04lx" params="prefix parent *origin min_angle:=1.5708 max_angle:=-1.5708">
+  <!--xacro:macro name="sensor_hokuyo_urg04lx" params="prefix parent *origin min_angle:=1.5708 max_angle:=-1.5708"-->
+  <xacro:macro name="sensor_hokuyo_urg04lx" params="prefix parent *origin min_angle:=2.36 max_angle:=-2.36">
     <joint name="${prefix}laser_joint" type="fixed">
       <!-- FRONT MOUNT  -->
@@ -45,5 +46,6 @@
 						<horizontal>
 							<!--samples>681</samples-->
-							<samples>180</samples>
+							<!--samples>180</samples-->
+							<samples>270</samples>
 							<resolution>1</resolution>
 							<min_angle>${min_angle}</min_angle>
@@ -52,5 +54,6 @@
 					</scan>
 					<range>
-						<min>0.02</min>
+						<!--min>0.02</min-->
+						<min>0.15</min>
 						<max>5.6</max>
 						<resolution>0.0061435</resolution>
