Commit message: gazebo ros control removed because was duplicated

File: turtlebot_description/urdf/sensors/rplidar.urdf.xacro (robot description, xacro)
@@ -15,7 +15,7 @@
       </collision>
       <visual>
-        <origin xyz="0 0 0" rpy="0 0 0"/>
+        <origin xyz="0 0 0" rpy="${-M_PI/2} 0 0"/>
         <geometry>
-            <mesh filename="package://turtlebot_description/meshes/sensors/rplidar.dae"/>
+            <mesh filename="package://turtlebot_description/meshes/sensors/rplidar2.dae"/>
         </geometry>
       </visual>
@@ -51,7 +51,7 @@
 					</scan>
 					<range>
-						<min>0.15</min>
-						<max>6.0</max>
-						<resolution>0.0174</resolution>
+						<min>0.25</min>
+						<max>10.0</max>
+						<resolution>0.000174</resolution>
 					</range>
 					<noise>

File: turtlebot_description/urdf/stacks/nostacks.gazebo.xacro (robot description, xacro)
@@ -5,5 +5,5 @@
         <!--robotNamespace>/rb1</robotNamespace-->
         <robotParam>robot_description</robotParam>
-        <controlPeriod>0.001</controlPeriod>
+        <controlPeriod>0.01</controlPeriod>
 	    <robotSimType>gazebo_ros_control/DefaultRobotHWSim</robotSimType>
       </plugin>

File: turtlebot_description/urdf/stacks/nostacks.urdf.xacro (robot description, xacro)
@@ -5,5 +5,5 @@
 <robot name="no_stacks" xmlns:xacro="http://ros.org/wiki/xacro">
   <xacro:include filename="$(find turtlebot_description)/urdf/common_properties.urdf.xacro"/>
-  <xacro:include filename="$(find turtlebot_description)/urdf/stacks/nostacks.gazebo.xacro"/>
+  <!--xacro:include filename="$(find turtlebot_description)/urdf/stacks/nostacks.gazebo.xacro"/-->
   <xacro:include filename="$(find turtlebot_description)/urdf/stacks/nostacks.transmission.xacro"/>
   <!-- Xacro properties -->
