Commit message: gazebo plugins updated

File: turtlebot_description/urdf/stacks/nostacks.gazebo.xacro (robot description, xacro)
@@ -1,4 +1,4 @@
 <?xml version="1.0"?>
-<robot xmlns:xacro="http://www.ros.org/wiki/xacro">
+<robot xmlns:xacro="http://ros.org/wiki/xacro">
 	<gazebo>
       <plugin name="ros_control" filename="libgazebo_ros_control.so">

File: turtlebot_description/urdf/stacks/nostacks.transmission.xacro (robot description, xacro)
@@ -1,4 +1,4 @@
 <?xml version="1.0"?>
-<robot xmlns:xacro="http://www.ros.org/wiki/xacro">
+<robot xmlns:xacro="http://ros.org/wiki/xacro">
 	<xacro:macro name="elevator_transmission" params="prefix_frame">
 	    <transmission name="${prefix_frame}plate_middle_transmission">

File: turtlebot_description/urdf/stacks/nostacks.urdf.xacro (robot description, xacro)
@@ -5,5 +5,5 @@
 <robot name="no_stacks" xmlns:xacro="http://ros.org/wiki/xacro">
   <xacro:include filename="$(find turtlebot_description)/urdf/common_properties.urdf.xacro"/>
-  <!--xacro:include filename="$(find turtlebot_description)/urdf/stacks/nostacks.gazebo.xacro"/-->
+  <xacro:include filename="$(find turtlebot_description)/urdf/stacks/nostacks.gazebo.xacro"/>
   <xacro:include filename="$(find turtlebot_description)/urdf/stacks/nostacks.transmission.xacro"/>
   <!-- Xacro properties -->
@@ -126,13 +126,13 @@
         <origin xyz="0.01364 0.0 0.0" rpy="0 0 0"/>
         <geometry>
-          <cylinder length="0.007" radius="0.170"/>
+          <cylinder length="0.007" radius="0.150"/>
         </geometry>
       </collision>
       <inertial>
-        <mass value="0.520" />
+        <mass value="0.0520" />
         <origin xyz="0 0 0" />
-        <inertia ixx="0.003328" ixy="0.0" ixz="0.0"
-                 iyy="0.003328" iyz="0.0"
-                 izz="0.006656" />
+        <inertia ixx="0.0003328" ixy="0.0" ixz="0.0"
+                 iyy="0.0003328" iyz="0.0"
+                 izz="0.0006656" />
       </inertial>
     </link>
