Commit message: Added prismatic joint

File: turtlebot_description/urdf/stacks/nostacks.urdf.xacro (robot description, xacro)
@@ -5,4 +5,6 @@
 <robot name="no_stacks" xmlns:xacro="http://ros.org/wiki/xacro">
   <xacro:include filename="$(find turtlebot_description)/urdf/common_properties.urdf.xacro"/>
+  <xacro:include filename="$(find turtlebot_description)/urdf/stacks/nostacks.gazebo.xacro"/>
+  <xacro:include filename="$(find turtlebot_description)/urdf/stacks/nostacks.transmission.xacro"/>
   <!-- Xacro properties -->
   <xacro:property name="M_SCALE" value="0.001"/>
@@ -92,5 +94,5 @@
         <origin xyz="-0.02364 0 0" rpy="0 0 0"/>
         <geometry>
-          <cylinder length="0.006" radius="0.170"/>
+          <cylinder length="0.007" radius="0.170"/>
         </geometry>
       </collision>
@@ -107,8 +109,10 @@
     <stack_middle_pole prefix_frame="${prefix_frame}" parent="${parent}" number="2" x_loc="-0.0381" y_loc= "0.1505" z_loc="0.1640"/>
     <stack_middle_pole prefix_frame="${prefix_frame}" parent="${parent}" number="3" x_loc="-0.0381" y_loc="-0.1505" z_loc="0.1640"/>
-    <joint name="${prefix_frame}plate_middle_joint" type="fixed">
-      <origin xyz="-0.01364 0.0 0.1874" rpy="0 0 0"/>
+    <joint name="${prefix_frame}plate_middle_joint" type="prismatic">
+      <origin xyz="-0.01364 0.0 0.1914" rpy="0 0 0"/>
       <parent link="${parent}"/>
       <child link="${prefix_frame}plate_middle_link"/>
+      <limit lower="0" upper="0.1" effort="1.0" velocity="0.5"/>
+      <axis xyz="0 0 1"/>
     </joint>
     <link name="${prefix_frame}plate_middle_link">
@@ -122,5 +126,5 @@
         <origin xyz="0.01364 0.0 0.0" rpy="0 0 0"/>
         <geometry>
-          <cylinder length="0.006" radius="0.170"/>
+          <cylinder length="0.007" radius="0.170"/>
         </geometry>
       </collision>
@@ -133,4 +137,5 @@
       </inertial>
     </link>
+    <xacro:elevator_transmission prefix_frame="${prefix_frame}" />
   </xacro:macro>
 </robot>

Commit message: turtlebot_description: friction added to middle plate

File: turtlebot_description/urdf/stacks/nostacks.urdf.xacro (robot description, xacro)
@@ -113,5 +113,5 @@
       <parent link="${parent}"/>
       <child link="${prefix_frame}plate_middle_link"/>
-      <limit lower="0" upper="0.1" effort="1.0" velocity="0.5"/>
+      <limit lower="0.0" upper="0.1" effort="1.0" velocity="0.05"/>
       <axis xyz="0 0 1"/>
     </joint>
@@ -137,5 +137,20 @@
       </inertial>
     </link>
-    <xacro:elevator_transmission prefix_frame="${prefix_frame}" />
+    <gazebo reference="${prefix_frame}plate_middle_link">
+    <collision name="${prefix_frame}plate_middle_link_collision">
+      <surface>
+        <friction>
+		  <ode>
+              <mu>1000</mu>
+              <mu2>1000</mu2>
+              <fdir1>0 0 0</fdir1>
+              <slip1>0</slip1>
+              <slip2>0</slip2>
+            </ode>
+        </friction>
+      </surface>
+    </collision>
+  </gazebo>
+  <xacro:elevator_transmission prefix_frame="${prefix_frame}" />
   </xacro:macro>
 </robot>
